File: pico-sdx/Oscillator.kicad_sch (KiCad schematic)
At the start: 1 part

Commit message: modular design
Connections:
- net +5VD renamed +3.3V
Changed lines of the file:
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@@
     )
   )
-  (symbol (lib_id "power:+5VD") (at 128.27 80.01 0) (unit 1)
+  (symbol (lib_id "power:+3.3V") (at 128.27 80.01 0) (unit 1)
     (in_bom yes) (on_board yes) (dnp no) (fields_autoplaced)
     (property "Reference" "#PWR067" (at 128.27 83.82 0)
       (effects (font (size 1.27 1.27)) hide)
     )
-    (property "Value" "+5VD" (at 128.27 74.93 0)
+    (property "Value" "+3.3V" (at 128.27 74.93 0)
       (effects (font (size 1.27 1.27)))
     )
