File: pico-sdx/power.kicad_sch (KiCad schematic)
At the start: 9 parts, among them U8 uA7805, U9 uA7805

Commit message: modular design
Connections:
- net +5VD renamed +3.3V
Changed lines of the file:
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@@
     )
   )
-  (symbol (lib_id "power:+5VD") (at 116.84 62.23 0) (unit 1)
+  (symbol (lib_id "power:+3.3V") (at 116.84 62.23 0) (unit 1)
     (in_bom yes) (on_board yes) (dnp no) (fields_autoplaced)
     (property "Reference" "#PWR060" (at 116.84 66.04 0)
       (effects (font (size 1.27 1.27)) hide)
     )
-    (property "Value" "+5VD" (at 116.84 57.15 0)
+    (property "Value" "+3.3V" (at 116.84 57.15 0)
       (effects (font (size 1.27 1.27)))
     )
