File: controller/controller.kicad_pcb (KiCad board)
At the start: 2 copper layers, 160 x 100 mm, 7 parts, among them J2 Barrel_Jack_Switch, J3 Conn_01x02, P1 PMOD-Device-x2-Type-Generic-A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, P2 PMOD-Device-x2-Type-Generic-A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, P3 PMOD-Device-x2-Type-Generic-A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, U3 ULN2803A

Commit message: remove external symbol and footprint libraries
Parts:
- A1: footprint crossover:ST_Zio_Connectors_144_STLink -> pico-sdx:ST_Zio_Connectors_144_STLink
Changed lines of the file:
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@@
 	(net 100 "unconnected-(A1D-D2{slash}PF15{slash}IO-PadCN10_12)")
 	(net 101 "unconnected-(A1C-D17{slash}PB15{slash}I2S_A_SD-PadCN7_3)")
-	(footprint "crossover:ST_Zio_Connectors_144_STLink"
+	(footprint "pico-sdx:ST_Zio_Connectors_144_STLink"
 		(layer "F.Cu")
 		(at 73.305 91.646 90)
@@
 			)
 		)
-		(property "Footprint" "crossover:ST_Zio_Connectors_144_STLink"
+		(property "Footprint" "pico-sdx:ST_Zio_Connectors_144_STLink"
 			(at 0 0 90)
 			(layer "F.Fab")
