File: mixer/buffer.kicad_sch (KiCad schematic)
At the start: 8 parts, among them U13 HMC589A

Commit message: add gerber export settings and get drc-clean
Parts:
- U13: symbol RF_Amplifier:HMC589A -> pico-sdx:HMC589A
Changed lines of the file:
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@@
 	)
 	(symbol
-		(lib_id "RF_Amplifier:HMC589A")
+		(lib_id "pico-sdx:HMC589A")
 		(at 124.46 66.04 0)
 		(unit 1)
