File: bandpass/bpf.kicad_sch (KiCad schematic)
At the start: 21 parts, among them K2 G6K-2, K3 G6K-2, K4 G6K-2, K5 G6K-2, K6 G6K-2, K7 G6K-2, K8 G6K-2, X1 40 m, X2 15 m, X3 30 m, X4 12 m, X5 20 m, X6 10 m, X7 17 m

Commit message: drc clean
Connections:
- net 10 m: now also D7.2 (A), K7.8; no longer D7.1 (K), K7.1
- net 12 m: now also D5.2 (A), K5.8; no longer D5.1 (K), K5.1
- net 15 m: now also D3.2 (A), K3.8; no longer D3.1 (K), K3.1
- net 17 m: now also D8.2 (A), K8.8; no longer D8.1 (K), K8.1
- net 20 m: now also D6.2 (A), K6.8; no longer D6.1 (K), K6.1
- net 30 m: now also D4.2 (A), K4.8; no longer D4.1 (K), K4.1
- net 40 m: now also D2.2 (A), K2.8; no longer D2.1 (K), K2.1
- net GND: no longer D2.2 (A), D3.2 (A), D4.2 (A), D5.2 (A), D6.2 (A), D7.2 (A), D8.2 (A), K2.8, K3.8, K4.8, K5.8, K6.8, K7.8, K8.8
- new net +12V: D2.1 (K), D3.1 (K), D4.1 (K), D5.1 (K), D6.1 (K), D7.1 (K), D8.1 (K), K2.1, K3.1, K4.1, K5.1, K6.1, K7.1, K8.1
