File: pa/pa.kicad_sch (KiCad schematic)
At the start: 63 parts, among them J1 Conn_01x02_Pin, J2 Conn_Coaxial, J3 Conn_Coaxial, P1 PMOD-Device-x2-Type-Generic-A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, Q1 Q_NMOS_GSD, Q2 Q_NMOS_GSD, Q3 IRLML6401, Q4 MMBT3904, T1 Transformer_1P_SS, T2 Transformer_1P_SS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

Commit message: replace 7806 by 1117
Parts:
- removed U1: L78L06_SO8, Package_SO:SOIC-8_3.9x4.9mm_P1.27mm, symbol Regulator_Linear:L78L06_SO8
- added R22, R23: R, Resistor_SMD:R_0603_1608Metric, symbol Device:R
- added U1: LT1117-ADJ, Package_TO_SOT_SMD:SOT-223-3_TabPin2, symbol Regulator_Linear:LT1117-ADJ
- J2, J3: footprint Connector_Coaxial:SMA_Amphenol_132289_EdgeMount -> Connector_Coaxial:SMA_Molex_73251-2200_Horizontal
Connections:
- net +12V: now also P1.12 (P12), P1.6 (P6); no longer C4.1, J1.1 (Pin_1), L1.2
- net +6V: now also R22.1, U1.2 (VO)
- net GND: now also R23.2
- net at C20.1, Q3.3 (D): now also U1.3 (VI)
- net +12VA renamed VDDA
- new net: R22.2, R23.1, U1.1 (ADJ)
- new net VDD: C4.1, J1.1 (Pin_1), L1.2
- no-connect marks 9 -> 7
Other:
- moved on the sheet: C17, C21

Commit message: drc clean
Parts:
- removed Q4: MMBT3904, Package_TO_SOT_SMD:SOT-23, symbol Transistor_BJT:MMBT3904
- removed R20: 1.8 kR, Resistor_SMD:R_1206_3216Metric, symbol Device:R
Connections:
- net TX~{RX}: now also R21.2
Changed lines of the file:
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@@
 	(wire
 		(pts
+			(xy 54.61 392.43) (xy 62.23 392.43)
+		)
+		(stroke
+			(width 0)
+			(type default)
+		)
+	)
+	(wire
+		(pts
 			(xy 76.2 377.19) (xy 62.23 377.19)
 		)
@@
 	(wire
 		(pts
+			(xy 62.23 392.43) (xy 62.23 388.62)
+		)
+		(stroke
+			(width 0)
+			(type default)
+		)
+	)
+	(wire
+		(pts
 			(xy 110.49 60.96) (xy 110.49 74.93)
 		)
@@
 	(global_label "TX~{RX}"
 		(shape input)
-		(at 46.99 393.7 180)
+		(at 54.61 392.43 180)
 		(fields_autoplaced yes)
 		(effects
@@
 		)
 		(property "Intersheetrefs" "${INTERSHEET_REFS}"
-			(at 39.3482 393.7 0)
+			(at 46.9682 392.43 0)
 			(effects
 				(font
@@
 	)
 	(symbol
-		(lib_id "power:GND")
-		(at 62.23 398.78 0)
-		(mirror y)
-		(unit 1)
-		(exclude_from_sim no)
-		(in_bom yes)
-		(on_board yes)
-		(dnp no)
-		(fields_autoplaced yes)
-		(property "Reference" "#PWR029"
-			(at 62.23 405.13 0)
-			(effects
-				(font
-					(size 1.27 1.27)
-				)
-				(hide yes)
-			)
-		)
-		(property "Value" "GND"
-			(at 62.23 403.86 0)
-			(effects
-				(font
-					(size 1.27 1.27)
-				)
-			)
-		)
-		(property "Footprint" ""
-			(at 62.23 398.78 0)
-			(effects
-				(font
-					(size 1.27 1.27)
-				)
-				(hide yes)
-			)
-		)
-		(property "Datasheet" ""
-			(at 62.23 398.78 0)
-			(effects
-				(font
-					(size 1.27 1.27)
-				)
-				(hide yes)
-			)
-		)
-		(property "Description" "Power symbol creates a global label with name \"GND\" , ground"
-			(at 62.23 398.78 0)
-			(effects
-				(font
-					(size 1.27 1.27)
-				)
-				(hide yes)
-			)
-		)
-		(pin "1"
-		)
-		(instances
-			(project "pa"
-				(path "/f9dbb021-4fea-4b33-8c2d-2c1606f600db"
-					(reference "#PWR029")
-					(unit 1)
-				)
-			)
-		)
-	)
-	(symbol
 		(lib_id "Device:R")
 		(at 68.58 54.61 180)
@@
 	)
 	(symbol
-		(lib_id "Device:R")
-		(at 50.8 393.7 90)
-		(unit 1)
-		(exclude_from_sim no)
-		(in_bom yes)
-		(on_board yes)
-		(dnp no)
-		(fields_autoplaced yes)
-		(property "Reference" "R20"
-			(at 50.8 387.35 90)
-			(effects
-				(font
-					(size 1.27 1.27)
-				)
-			)
-		)
-		(property "Value" "1.8 kR"
-			(at 50.8 389.89 90)
-			(effects
-				(font
-					(size 1.27 1.27)
-				)
-			)
-		)
-		(property "Footprint" "Resistor_SMD:R_1206_3216Metric"
-			(at 50.8 395.478 90)
-			(effects
-				(font
-					(size 1.27 1.27)
-				)
-				(hide yes)
-			)
-		)
-		(property "Datasheet" "~"
-			(at 50.8 393.7 0)
-			(effects
-				(font
-					(size 1.27 1.27)
-				)
-				(hide yes)
-			)
-		)
-		(property "Description" "Resistor"
-			(at 50.8 393.7 0)
-			(effects
-				(font
-					(size 1.27 1.27)
-				)
-				(hide yes)
-			)
-		)
-		(pin "1"
-		)
-		(pin "2"
-		)
-		(instances
-			(project "pa"
-				(path "/f9dbb021-4fea-4b33-8c2d-2c1606f600db"
-					(reference "R20")
-					(unit 1)
-				)
-			)
-		)
-	)
-	(symbol
 		(lib_id "power:PWR_FLAG")
 		(at 175.26 153.67 0)
@@
 					(unit 1)
 				)
-			)
-		)
-	)
-	(symbol
-		(lib_id "Transistor_BJT:MMBT3904")
-		(at 59.69 393.7 0)
-		(unit 1)
-		(exclude_from_sim no)
-		(in_bom yes)
-		(on_board yes)
-		(dnp no)
-		(fields_autoplaced yes)
-		(property "Reference" "Q4"
-			(at 64.77 392.4299 0)
-			(effects
-				(font
-					(size 1.27 1.27)
-				)
-				(justify left)
-			)
-		)
-		(property "Value" "MMBT3904"
-			(at 64.77 394.9699 0)
-			(effects
-				(font
-					(size 1.27 1.27)
-				)
-				(justify left)
-			)
-		)
-		(property "Footprint" "Package_TO_SOT_SMD:SOT-23"
-			(at 64.77 395.605 0)
-			(effects
-				(font
-					(size 1.27 1.27)
-					(italic yes)
-				)
-				(justify left)
-				(hide yes)
-			)
-		)
-		(property "Datasheet" "https://www.onsemi.com/pdf/datasheet/pzt3904-d.pdf"
-			(at 59.69 393.7 0)
-			(effects
-				(font
-					(size 1.27 1.27)
-				)
-				(justify left)
-				(hide yes)
-			)
-		)
-		(property "Description" "0.2A Ic, 40V Vce, Small Signal NPN Transistor, SOT-23"
-			(at 59.69 393.7 0)
-			(effects
-				(font
-					(size 1.27 1.27)
-				)
-				(hide yes)
-			)
-		)
-		(pin "2"
-		)
-		(pin "1"
-		)
-		(pin "3"
-		)
-		(instances
-			(project ""
-				(path "/f9dbb021-4fea-4b33-8c2d-2c1606f600db"
-					(reference "Q4")
-					(unit 1)
-				)
